File: electrical/head.brd (EAGLE design)
At the start: 60 x 100 mm, 34 parts, among them Q1 N-FET, U1 TEENSY_3.1-3.2_OUTER_ROW, U2 USB2514BI

Commit message: head circuit WIP
Parts:
- removed USB-UPSTREAM: (no value), bleed:JST-3-PTH
- added C16, C17, C18, C19, C20, C21: (no value), bleed:EIA3216-KIT
- added C22, C23: (no value), bleed:CPOL-RADIAL-1000UF-25V
- added D2, D3: (no value), bleed:SMA-DIODE-KIT
- added IC2, IC3: (no value), bleed:SOT23
- added JP1: (no value), bleed:MOLEX-1X4
- added JP2: (no value), bleed:1X10
- added JP3: (no value), bleed:MOLEX-1X2
- added JP4: (no value), bleed:JST-2-PTH
- added LED1, LED2, LED3, LED4: (no value), bleed:LED-0603
- added Q2: N-FET, bleed:TO220V
- added Q3: N-FET, bleed:SOT23-3
- added R10, R11, R12, R13, R14, R8, R9: (no value), bleed:0603-RES
- added R7: (no value), bleed:0402-RES
- added S1: SLOW-FIRE, bleed:TACTILE-SWITCH-1101NE
- added TVS1, TVS2, TVS3: TVS-SOD323, bleed:SOD-323
- added X1, X2, X3, X4, X5: USB-JSTXH-VERT-TH, bleed:1X04-JSTXH-VERT-TH
- U1: value TEENSY_3.1-3.2_OUTER_ROW -> TEENSY-3.2
- moved IC1 47.4 mm to (54.5, 39.5), turned to 180 degrees
- moved C2 45.6 mm to (49.5, 43.0), flipped to the bottom
- moved R1 24.4 mm to (37.5, 63.0)
- moved C1 21.8 mm to (46.0, 39.5)
- moved R2 20.8 mm to (35.5, 63.0)
- moved Q1 6.52 mm to (40.5, 66.5), turned to 0 degrees
- moved C3 3.50 mm to (44.0, 54.5)
- moved D1 3.50 mm to (48.0, 64.0)
- moved C10 1.00 mm to (38.3, 10.7)
- moved C11 1.00 mm to (41.5, 12.1)
- moved C12 1.00 mm to (35.7, 12.0)
- moved C13 1.00 mm to (47.0, 13.9)
- moved C14 1.00 mm to (48.5, 13.9)
- moved C15 1.00 mm to (35.7, 10.5)
- moved C4 1.00 mm to (49.8, 7.40)
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Connections:
- removed net N$11: U2.2
- removed net N$17: U2.3
- removed net N$18: U2.7
- removed net N$20: U2.6
- removed net VIN: U1.VIN
- new net GUN-PWM: LED2.A, R1.1, R2.2, U1.23/A9
- new net HOPPER: LED3.A, R8.1, R9.2, U1.22/A8
- new net IMU-CS: JP2.9, U1.9
- new net IMU-INT: JP2.8, U1.10
- new net LASER: LED4.A, R10.2, R11.2, U1.21/A7
- new net N$10: IC3.2, JP4.2
- new net N$7: D2.A, JP3.1, Q2.2
- new net N$8: Q2.1, R8.2, TVS2.2
- new net N$9: JP4.1, Q3.3
- new net SERVO-DAC: JP1.4, U1.RESET/DAC
- new net SERVO-PULSE: JP1.3, U1.20/A6
- new net SLOW-FIRE: S1.P$1, U1.2
- new net SPI-MISO: JP2.7, U1.12
- new net SPI-MOSI: JP2.4, U1.11
- new net SPI-SCLK: JP2.3, U1.14/A0
- new net USB_DOWN1_D_N: U2.1, X5.3
- new net USB_DOWN1_D_P: U2.2, X5.2
- new net USB_DOWN2_D_N: U2.3, X4.3
- new net USB_DOWN2_D_P: U2.4, X4.2
- new net USB_DOWN3_D_N: U2.6, X3.3
- new net USB_DOWN3_D_P: U2.7, X3.2
- new net USB_DOWN4_D_N: U2.8, X2.3
- new net USB_DOWN4_D_P: U2.9, X2.2
- new net USB_UP_D_N: U2.31, X1.2
- new net USB_UP_D_P: U2.30, X1.3
- net +9V: now also C22.1, C23.1, D2.C, D3.C, JP1.2, JP3.2
- net 3.3V: now also C20.A, IC2.2, LED1.A
- net 5V: now also C16.A, C17.A, C18.A, C19.A, C21.A, D3.A, IC2.3, IC3.3, JP2.1, U1.VIN, X1.1, X2.1, X3.1, X4.1, X5.1
- net GND: now also C16.C, C17.C, C18.C, C19.C, C20.C, C21.C, C22.2, C23.2, IC2.1, IC3.1, JP1.1, JP2.10, JP2.2, Q2.3, Q3.2, R11.1, R12.1, R13.1, R14.1, R7.1, R9.1, S1.P$2, TVS1.1, TVS2.1, TVS3.1, X1.4, X2.4, X3.4, X4.4, X5.4; no longer USB-UPSTREAM.1
- net N$12: now also LED2.C, R12.2; no longer U2.1
- net N$13: now also Q3.1, R10.1, TVS3.2; no longer U2.30, USB-UPSTREAM.3
- net N$14: now also LED3.C, R13.2; no longer U2.31, USB-UPSTREAM.2
- net N$16: now also LED4.C, R14.2; no longer U2.4
- net N$3: now also LED1.C, R7.2; no longer R1.1, R2.2
- net N$4: now also TVS1.2
Routing:
- net +9V: track 0.00 -> 185.1 mm
- net 5V: track 0.00 -> 139.0 mm, vias 0 -> 1
- net SPI-SCLK: track 0.00 -> 51.9 mm, vias 0 -> 1
- net GUN-PWM: track 0.00 -> 48.1 mm
- net HOPPER: track 0.00 -> 42.0 mm
- net LASER: track 0.00 -> 37.5 mm
- net SPI-MOSI: track 0.00 -> 33.1 mm
- net SLOW-FIRE: track 0.00 -> 27.3 mm
- net SPI-MISO: track 0.00 -> 26.4 mm
- net USB_DOWN1_D_P: track 0.00 -> 22.9 mm
- net USB_DOWN1_D_N: track 0.00 -> 22.2 mm
- net IMU-INT: track 0.00 -> 21.3 mm, vias 0 -> 1
- net USB_DOWN4_D_N: track 0.00 -> 20.0 mm
- net USB_UP_D_N: track 0.00 -> 19.9 mm
- net USB_UP_D_P: track 0.00 -> 19.9 mm
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Other:
- board size 60 x 100 mm -> 60 x 70 mm

Commit message: head circuit WIP
Parts:
- removed BATT, GUN: (no value), bleed:TERMBLOCK-X2-OSTTF020161
- added JP5: (no value), bleed:1X10
- added LOGO1: LOGO_BLEED, bleed:LOGO_BLEED
- added SERVO: (no value), bleed:MOLEX-1X4
- C1, C2: device bleed:EIA3216-KIT -> bleed:CPOL-RADIAL-1000UF-25V
- C10, C11, C4, C5, C6, C7, C8, C9: device bleed:0402-CAP -> bleed:EIA3216-KIT
- C12, C14: value 100n -> (none)
- C13, C15: value 10n -> (none)
- C16, C17, C18, C19: device bleed:EIA3216-KIT -> bleed:0402-CAP
- C20: value (none) -> 100n; device bleed:EIA3216-KIT -> bleed:0402-CAP
- C21: value (none) -> 10n; device bleed:EIA3216-KIT -> bleed:0402-CAP
- C22: value (none) -> 100n; device bleed:CPOL-RADIAL-1000UF-25V -> bleed:0402-CAP
- C23: value (none) -> 10n; device bleed:CPOL-RADIAL-1000UF-25V -> bleed:0402-CAP
- IC1: value (none) -> +5V0
- IC2: value (none) -> +3V3
- IC3: value (none) -> +3V0
- JP1: device bleed:MOLEX-1X4 -> bleed:TERMBLOCK-X2-OSTTF020161
- JP2: device bleed:1X10 -> bleed:TERMBLOCK-X2-OSTTF020161
- R10, R11, R12, R13: device bleed:0603-RES -> bleed:0402-RES
- R14: value (none) -> 12K; device bleed:0603-RES -> bleed:0402-RES
- R3: value 12K -> (none); device bleed:0402-RES -> bleed:0603-RES
- R4, R5, R6, R7: device bleed:0402-RES -> bleed:0603-RES
- TVS1, TVS2, TVS3: value TVS-SOD323 -> (none)
- Y1: value (none) -> 24MHz
- moved SCREW4 69.7 mm to (57.0, 3.00)
- moved R7 63.7 mm to (31.0, 64.5), turned to 0 degrees
- moved R12 61.9 mm to (44.3, 4.00), turned to 90 degrees
- moved R10 61.4 mm to (49.5, 3.50), turned to 270 degrees
- moved LED1 61.4 mm to (33.0, 63.0), turned to 90 degrees
- moved R5 59.4 mm to (24.5, 60.0), turned to 270 degrees
- moved R4 59.3 mm to (35.5, 63.0), turned to 270 degrees
- moved JP2 57.8 mm to (55.5, 65.0), turned to 0 degrees
- moved JP1 57.7 mm to (55.0, 54.5)
- moved LED4 57.3 mm to (48.0, 3.50), turned to 180 degrees
- moved R6 55.7 mm to (12.5, 50.5), turned to 180 degrees
- moved R11 55.0 mm to (41.9, 4.00), turned to 90 degrees
- moved SCREW3 54.0 mm to (3.00, 47.0)
- moved R13 51.5 mm to (43.1, 4.00)
- moved R3 50.0 mm to (12.5, 52.5), turned to 180 degrees
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Connections:
- removed net N$12 (its old number): LED2.C, R12.2
- new net N$3: LED4.C, R10.2
- net +9V: now also C1.1, C2.1, C4.A, JP2.2, SERVO.2; no longer BATT.2, C2.A, C22.1, C23.1, GUN.2
- net 3.3V: now also C12.2, C13.2, C14.2, C15.2, C16.2, C17.2, C9.A, LED4.A, R13.1; no longer C10.2, C11.2, C20.A, C6.2, C7.2, C8.2, C9.2, LED1.A, R6.1
- net 5V: now also C10.A, C11.A, C5.A, C6.A, C7.A, C8.A, D1.A, JP5.1; no longer C1.A, C16.A, C17.A, C18.A, C19.A, C21.A, D3.A, JP2.1
- net GND: now also C1.2, C10.C, C11.C, C16.1, C17.1, C18.1, C19.1, C2.2, C20.1, C21.1, C22.1, C23.1, C4.C, C5.C, C6.C, C7.C, C8.C, C9.C, JP5.10, JP5.2, R10.1, R6.1, R8.1, S1.2, SERVO.1; no longer BATT.1, C1.C, C10.1, C11.1, C16.C, C17.C, C18.C, C19.C, C2.C, C20.C, C21.C, C22.2, C23.2, C4.1, C5.1, C6.1, C7.1, C8.1, C9.1, JP2.10, JP2.2, R13.1, R2.1, R3.1, S1.P$2
- net GUN-PWM: now also LED1.A, R4.2; no longer LED2.A, R2.2
- net HOPPER: now also LED2.A, R2.1, R5.2; no longer LED3.A, R8.1, R9.2
- net HUB-RST: now also R13.2; no longer R6.2
- net IMU-CS: now also JP5.9; no longer JP2.9
- net IMU-INT: now also JP5.8; no longer JP2.8
- net LASER: now also LED3.A, R3.2, R6.2; no longer LED4.A, R10.2, R11.2
- net N$1: now also C18.2; no longer C4.2
- net N$13: now also R3.1; no longer R10.1
- net N$14: now also LED2.C, R8.2; no longer LED3.C, R13.2
- net N$15: now also C22.2, C23.2; no longer C12.2, C15.2
- net N$16: now also LED3.C, R9.2; no longer LED4.C, R14.2
- net N$19: now also R14.2; no longer R3.2
- net N$2: now also D2.A, JP2.1; no longer D1.A, GUN.1
- net N$21: now also R11.2; no longer R4.2
- net N$22: now also R12.2; no longer R5.2
- net N$5: now also C19.2; no longer C5.2
- net N$6: now also C20.2, C21.2; no longer C13.2, C14.2
- net N$7: now also D3.A; no longer D2.A
- net N$8: now also R2.2; no longer R8.2
- net SERVO-DAC: now also SERVO.4; no longer JP1.4
- net SERVO-PULSE: now also SERVO.3; no longer JP1.3
- net SLOW-FIRE: now also S1.1; no longer S1.P$1
- net SPI-MISO: now also JP5.7; no longer JP2.7
- net SPI-MOSI: now also JP5.4; no longer JP2.4
- net SPI-SCLK: now also JP5.3; no longer JP2.3
- net USB_DOWN1_D_N: now also X4.3; no longer X5.3
- net USB_DOWN1_D_P: now also X4.2; no longer X5.2
- net USB_DOWN2_D_N: now also X3.3; no longer X4.3
- net USB_DOWN2_D_P: now also X3.2; no longer X4.2
- net USB_DOWN3_D_N: now also X2.3; no longer X3.3
- net USB_DOWN3_D_P: now also X2.2; no longer X3.2
- net USB_DOWN4_D_N: now also X1.3; no longer X2.3
- net USB_DOWN4_D_P: now also X1.2; no longer X2.2
- net USB_UP_D_N: now also X5.2; no longer X1.2
- net USB_UP_D_P: now also X5.3; no longer X1.3
Routing:
- net +9V: track 185.1 -> 192.1 mm
- net N$12 (its old number): track 1.90 -> 0.00 mm
- net SPI-SCLK: track 51.9 -> 50.2 mm, vias 1 -> 0
- net SERVO-DAC: track 16.3 -> 18.0 mm
- net N$3: track 0.00 -> 1.54 mm
- net N$2: track 19.1 -> 18.2 mm
- net GND: vias 78 -> 99
Other:
- board text added: "GUN"
- board text added: "PWR"
