File: electrical/head.sch (EAGLE design)
At the start: 34 parts, among them Q1 N-FET, U1 TEENSY_3.1-3.2_OUTER_ROW, U2 USB2514BI

Commit message: head circuit WIP
Parts:
- removed USB-UPSTREAM: (no value), bleed:M03JST-PTH
- added C16, C17, C18, C19, C20, C21: (no value), bleed:CAP_POL1206-KIT
- added C22, C23: (no value), bleed:CAP_POLPTH4
- added D2, D3: (no value), bleed:DIODESMA-KIT
- added IC2, IC3: (no value), bleed:V_REG_78XX-SOT23
- added JP1: (no value), bleed:M04POLAR
- added JP2: M10", bleed:M10"
- added JP3: (no value), bleed:M02POLAR
- added JP4: (no value), bleed:M02JST-PTH-2
- added LED1, LED2, LED3, LED4: (no value), bleed:LED0603
- added Q2: N-FET, bleed:MOSFET-NCHANNELPTH2
- added Q3: N-FET, bleed:MOSFET-NCHANNELSMD
- added R10, R11, R12, R13, R14, R8, R9: (no value), bleed:RESISTOR0603-RES
- added R7: (no value), bleed:RESISTOR0402-RES
- added S1: SLOW-FIRE, bleed:SWITCH-MOMENTARY-2-SMD-1101NE
- added TVS1, TVS2, TVS3: TVS-SOD323, bleed:TVS-SOD323
- added X1, X2, X3, X4, X5: USB-JSTXH-VERT-TH, bleed:USB-JSTXH-VERT-TH
- U1: value TEENSY_3.1-3.2_OUTER_ROW -> TEENSY-3.2
Connections:
- removed net N$11: U2.USB-DP-1
- removed net N$17: U2.USB-DM-2
- removed net N$18: U2.USB-DP-3
- removed net N$20: U2.USB-DM-3
- new net GUN-PWM: LED2.A, R1.1, R2.2, U1.23/A9/T/PWM
- new net HOPPER: LED3.A, R8.1, R9.2, U1.22/A8/T/PWM
- new net IMU-CS: JP2.9, U1.9/RX2/PWM/(CS)
- new net IMU-INT: JP2.8, U1.10/TX2/PWM/CS
- new net LASER: LED4.A, R10.2, R11.2, U1.21/A7/PWM/(RX1)/(CS)
- new net N$10: IC3.OUT, JP4.2
- new net N$7: D2.A, JP3.1, Q2.D
- new net N$8: Q2.G, R8.2, TVS2.2
- new net N$9: JP4.1, Q3.D
- new net SERVO-DAC: JP1.4, U1.A14/DAC
- new net SERVO-PULSE: JP1.3, U1.20/A6/PWM/(CS)
- new net SLOW-FIRE: S1.1, U1.2
- new net SPI-MISO: JP2.7, U1.12/MISO
- new net SPI-MOSI: JP2.4, U1.11/MOSI
- new net SPI-SCLK: JP2.3, U1.14/A0/(SCK)
- new net USB_DOWN1_D_N: U2.USB-DM-1, X5.D-
- new net USB_DOWN1_D_P: U2.USB-DP-1, X5.D+
- new net USB_DOWN2_D_N: U2.USB-DM-2, X4.D-
- new net USB_DOWN2_D_P: U2.USB-DP-2, X4.D+
- new net USB_DOWN3_D_N: U2.USB-DM-3, X3.D-
- new net USB_DOWN3_D_P: U2.USB-DP-3, X3.D+
- new net USB_DOWN4_D_N: U2.USB-DM-4, X2.D-
- new net USB_DOWN4_D_P: U2.USB-DP-4, X2.D+
- new net USB_UP_D_N: U2.USB-DP-UP, X1.D+
- new net USB_UP_D_P: U2.USB-DM-UP, X1.D-
- net +9V: now also C22.+, C23.+, D2.C, D3.C, JP1.2, JP3.2
- net 3.3V: now also C20.+, IC2.OUT, LED1.A
- net 5V: now also C16.+, C17.+, C18.+, C19.+, C21.+, D3.A, IC2.IN, IC3.IN, JP2.1, U1.VIN, X1.VBUS, X2.VBUS, X3.VBUS, X4.VBUS, X5.VBUS
- net GND: now also C16.-, C17.-, C18.-, C19.-, C20.-, C21.-, C22.-, C23.-, IC2.GND, IC3.GND, JP1.1, JP2.10, JP2.2, Q2.S, Q3.S, R11.1, R12.1, R13.1, R14.1, R7.1, R9.1, S1.2, TVS1.1, TVS2.1, TVS3.1, X1.GND, X2.GND, X3.GND, X4.GND, X5.GND; no longer USB-UPSTREAM.1
- net N$12: now also LED2.C, R12.2; no longer U2.USB-DM-1
- net N$13: now also Q3.G, R10.1, TVS3.2; no longer U2.USB-DM-UP, USB-UPSTREAM.3
- net N$14: now also LED3.C, R13.2; no longer U2.USB-DP-UP, USB-UPSTREAM.2
- net N$16: now also LED4.C, R14.2; no longer U2.USB-DP-2
- net N$3: now also LED1.C, R7.2; no longer R1.1, R2.2
- net N$4: now also TVS1.2
Other:
- moved on the sheet: R1, R2

Commit message: head circuit WIP
Parts:
- removed BATT, GUN: (no value), bleed:M02-TERMBLOCK-3.5MM-OSTTF020161
- added JP5: M10", bleed:M10"
- added LOGO1: LOGO_BLEED, bleed:LOGO_BLEED
- added SERVO: (no value), bleed:M04POLAR
- C1, C2: device bleed:CAP_POL1206-KIT -> bleed:CAP_POLPTH4
- C10, C11, C4, C5, C6, C7, C8, C9: device bleed:CAP0402-CAP -> bleed:CAP_POL1206-KIT
- C12, C14: value 100n -> (none)
- C13, C15: value 10n -> (none)
- C16, C17, C18, C19: device bleed:CAP_POL1206-KIT -> bleed:CAP0402-CAP
- C20: value (none) -> 100n; device bleed:CAP_POL1206-KIT -> bleed:CAP0402-CAP
- C21: value (none) -> 10n; device bleed:CAP_POL1206-KIT -> bleed:CAP0402-CAP
- C22: value (none) -> 100n; device bleed:CAP_POLPTH4 -> bleed:CAP0402-CAP
- C23: value (none) -> 10n; device bleed:CAP_POLPTH4 -> bleed:CAP0402-CAP
- IC1: value (none) -> +5V0
- IC2: value (none) -> +3V3
- IC3: value (none) -> +3V0
- JP1: device bleed:M04POLAR -> bleed:M02-TERMBLOCK-3.5MM-OSTTF020161
- JP2: value M10" -> (none); device bleed:M10" -> bleed:M02-TERMBLOCK-3.5MM-OSTTF020161
- R10, R11, R12, R13: device bleed:RESISTOR0603-RES -> bleed:RESISTOR0402-RES
- R14: value (none) -> 12K; device bleed:RESISTOR0603-RES -> bleed:RESISTOR0402-RES
- R3: value 12K -> (none); device bleed:RESISTOR0402-RES -> bleed:RESISTOR0603-RES
- R4, R5, R6, R7: device bleed:RESISTOR0402-RES -> bleed:RESISTOR0603-RES
- Y1: value (none) -> 24MHz
Connections:
- removed net N$12 (its old number): LED2.C, R12.2
- new net N$3: LED4.C, R10.2
- net +9V: now also C1.+, C4.+, JP2.2, SERVO.2; no longer BATT.2, C22.+, C23.+, GUN.2
- net 3.3V: now also C12.2, C13.2, C14.2, C15.2, C16.2, C17.2, C9.+, LED4.A, R13.1; no longer C10.2, C11.2, C20.+, C6.2, C7.2, C8.2, C9.2, LED1.A, R6.1
- net 5V: now also C10.+, C11.+, C5.+, C6.+, C7.+, C8.+, D1.A, JP5.1; no longer C1.+, C16.+, C17.+, C18.+, C19.+, C21.+, D3.A, JP2.1
- net GND: now also C10.-, C11.-, C16.1, C17.1, C18.1, C19.1, C20.1, C21.1, C22.1, C23.1, C4.-, C5.-, C6.-, C7.-, C8.-, C9.-, JP5.10, JP5.2, R10.1, R6.1, R8.1, SERVO.1; no longer BATT.1, C10.1, C11.1, C16.-, C17.-, C18.-, C19.-, C20.-, C21.-, C22.-, C23.-, C4.1, C5.1, C6.1, C7.1, C8.1, C9.1, JP2.10, JP2.2, R13.1, R2.1, R3.1
- net GUN-PWM: now also LED1.A, R4.2; no longer LED2.A, R2.2
- net HOPPER: now also LED2.A, R2.1, R5.2; no longer LED3.A, R8.1, R9.2
- net HUB-RST: now also R13.2; no longer R6.2
- net IMU-CS: now also JP5.9; no longer JP2.9
- net IMU-INT: now also JP5.8; no longer JP2.8
- net LASER: now also LED3.A, R3.2, R6.2; no longer LED4.A, R10.2, R11.2
- net N$1: now also C18.2; no longer C4.2
- net N$13: now also R3.1; no longer R10.1
- net N$14: now also LED2.C, R8.2; no longer LED3.C, R13.2
- net N$15: now also C22.2, C23.2; no longer C12.2, C15.2
- net N$16: now also LED3.C, R9.2; no longer LED4.C, R14.2
- net N$19: now also R14.2; no longer R3.2
- net N$2: now also D2.A, JP2.1; no longer D1.A, GUN.1
- net N$21: now also R11.2; no longer R4.2
- net N$22: now also R12.2; no longer R5.2
- net N$5: now also C19.2; no longer C5.2
- net N$6: now also C20.2, C21.2; no longer C13.2, C14.2
- net N$7: now also D3.A; no longer D2.A
- net N$8: now also R2.2; no longer R8.2
- net SERVO-DAC: now also SERVO.4; no longer JP1.4
- net SERVO-PULSE: now also SERVO.3; no longer JP1.3
- net SPI-MISO: now also JP5.7; no longer JP2.7
- net SPI-MOSI: now also JP5.4; no longer JP2.4
- net SPI-SCLK: now also JP5.3; no longer JP2.3
- net USB_DOWN1_D_N: now also X4.D-; no longer X5.D-
- net USB_DOWN1_D_P: now also X4.D+; no longer X5.D+
- net USB_DOWN2_D_N: now also X3.D-; no longer X4.D-
- net USB_DOWN2_D_P: now also X3.D+; no longer X4.D+
- net USB_DOWN3_D_N: now also X2.D-; no longer X3.D-
- net USB_DOWN3_D_P: now also X2.D+; no longer X3.D+
- net USB_DOWN4_D_N: now also X1.D-; no longer X2.D-
- net USB_DOWN4_D_P: now also X1.D+; no longer X2.D+
- net USB_UP_D_N: now also X5.D+; no longer X1.D+
- net USB_UP_D_P: now also X5.D-; no longer X1.D-
Other:
- moved on the sheet: C1, C12, C13, C14, C15, C2, C3, D1, D2, D3, IC1, IC2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
